Commit message: change vis_utils

File: retarget_wmq/urdf/allegro_hand_left_glb.urdf (robot description, URDF)
Before this commit: robot allegro_left, 29 links, 28 joints
Links:
- link base_link: geometry collision box size=0.0414 0.0538 0.0428; collision box size=0.0414 0.072 0.013
- link link_0.0: geometry collision box size=0.0196 0.0275 0.0164; visual mesh filename=/home/wangminqi/workspace/test/packages/hands/allegro_hand/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
- link link_1.0: geometry collision box size=0.0196 0.0275 0.054; visual mesh filename=/home/wangminqi/workspace/test/packages/hands/allegro_hand/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
- link link_10.0: geometry collision box size=0.0196 0.0275 0.0384; visual mesh filename=/home/wangminqi/workspace/test/packages/hands/allegro_hand/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
- link link_11.0: geometry collision box size=0.0196 0.0269 0.022; visual mesh filename=/home/wangminqi/workspace/test/packages/hands/allegro_hand/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
- link link_11.0_tip: geometry collision mesh filename=/home/wangminqi/workspace/test/packages/hands/allegro_hand/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; visual mesh filename=/home/wangminqi/workspace/test/packages/hands/allegro_hand/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
- link link_12.0: geometry collision box size=0.0358 0.034 0.0455; visual mesh filename=/home/wangminqi/workspace/test/packages/hands/allegro_hand/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
- link link_13.0: geometry collision box size=0.0196 0.0275 0.0177; visual mesh filename=/home/wangminqi/workspace/test/packages/hands/allegro_hand/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
- link link_14.0: geometry collision box size=0.0196 0.0275 0.0514; visual mesh filename=/home/wangminqi/workspace/test/packages/hands/allegro_hand/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
- link link_15.0: geometry collision box size=0.0196 0.0269 0.04; visual mesh filename=/home/wangminqi/workspace/test/packages/hands/allegro_hand/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
- link link_15.0_tip: geometry collision mesh filename=/home/wangminqi/workspace/test/packages/hands/allegro_hand/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; visual mesh filename=/home/wangminqi/workspace/test/packages/hands/allegro_hand/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
- link link_2.0: geometry collision box size=0.0196 0.0275 0.0384; visual mesh filename=/home/wangminqi/workspace/test/packages/hands/allegro_hand/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
- link link_3.0: geometry collision box size=0.0196 0.0269 0.022; visual mesh filename=/home/wangminqi/workspace/test/packages/hands/allegro_hand/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
- link link_3.0_tip: geometry collision mesh filename=/home/wangminqi/workspace/test/packages/hands/allegro_hand/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; visual mesh filename=/home/wangminqi/workspace/test/packages/hands/allegro_hand/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
- link link_4.0: geometry collision box size=0.0196 0.0275 0.0164; visual mesh filename=/home/wangminqi/workspace/test/packages/hands/allegro_hand/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
- link link_5.0: geometry collision box size=0.0196 0.0275 0.054; visual mesh filename=/home/wangminqi/workspace/test/packages/hands/allegro_hand/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
- link link_6.0: geometry collision box size=0.0196 0.0275 0.0384; visual mesh filename=/home/wangminqi/workspace/test/packages/hands/allegro_hand/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
- link link_7.0: geometry collision box size=0.0196 0.0269 0.022; visual mesh filename=/home/wangminqi/workspace/test/packages/hands/allegro_hand/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
- link link_7.0_tip: geometry collision mesh filename=/home/wangminqi/workspace/test/packages/hands/allegro_hand/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; visual mesh filename=/home/wangminqi/workspace/test/packages/hands/allegro_hand/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
- link link_8.0: geometry collision box size=0.0196 0.0275 0.0164; visual mesh filename=/home/wangminqi/workspace/test/packages/hands/allegro_hand/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
- link link_9.0: geometry collision box size=0.0196 0.0275 0.054; visual mesh filename=/home/wangminqi/workspace/test/packages/hands/allegro_hand/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

File: retarget_wmq/urdf/allegro_hand_right_glb.urdf (robot description, URDF)
Before this commit: robot allegro_right, 29 links, 28 joints
Links:
- link base_link: geometry collision box size=0.0414 0.0538 0.0428; collision box size=0.0414 0.072 0.013
- link link_0.0: geometry collision box size=0.0196 0.0275 0.0164; visual mesh filename=/home/wangminqi/workspace/test/packages/hands/allegro_hand/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
- link link_1.0: geometry collision box size=0.0196 0.0275 0.054; visual mesh filename=/home/wangminqi/workspace/test/packages/hands/allegro_hand/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
- link link_10.0: geometry collision box size=0.0196 0.0275 0.0384; visual mesh filename=/home/wangminqi/workspace/test/packages/hands/allegro_hand/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
- link link_11.0: geometry collision box size=0.0196 0.0269 0.022; visual mesh filename=/home/wangminqi/workspace/test/packages/hands/allegro_hand/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
- link link_11.0_tip: geometry collision mesh filename=/home/wangminqi/workspace/test/packages/hands/allegro_hand/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; visual mesh filename=/home/wangminqi/workspace/test/packages/hands/allegro_hand/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
- link link_12.0: geometry collision box size=0.0358 0.034 0.0455; visual mesh filename=/home/wangminqi/workspace/test/packages/hands/allegro_hand/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
- link link_13.0: geometry collision box size=0.0196 0.0275 0.0177; visual mesh filename=/home/wangminqi/workspace/test/packages/hands/allegro_hand/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
- link link_14.0: geometry collision box size=0.0196 0.0275 0.0514; visual mesh filename=/home/wangminqi/workspace/test/packages/hands/allegro_hand/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
- link link_15.0: geometry collision box size=0.0196 0.0269 0.04; visual mesh filename=/home/wangminqi/workspace/test/packages/hands/allegro_hand/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
- link link_15.0_tip: geometry collision mesh filename=/home/wangminqi/workspace/test/packages/hands/allegro_hand/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; visual mesh filename=/home/wangminqi/workspace/test/packages/hands/allegro_hand/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
- link link_2.0: geometry collision box size=0.0196 0.0275 0.0384; visual mesh filename=/home/wangminqi/workspace/test/packages/hands/allegro_hand/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
- link link_3.0: geometry collision box size=0.0196 0.0269 0.022; visual mesh filename=/home/wangminqi/workspace/test/packages/hands/allegro_hand/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
- link link_3.0_tip: geometry collision mesh filename=/home/wangminqi/workspace/test/packages/hands/allegro_hand/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; visual mesh filename=/home/wangminqi/workspace/test/packages/hands/allegro_hand/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
- link link_4.0: geometry collision box size=0.0196 0.0275 0.0164; visual mesh filename=/home/wangminqi/workspace/test/packages/hands/allegro_hand/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
- link link_5.0: geometry collision box size=0.0196 0.0275 0.054; visual mesh filename=/home/wangminqi/workspace/test/packages/hands/allegro_hand/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
- link link_6.0: geometry collision box size=0.0196 0.0275 0.0384; visual mesh filename=/home/wangminqi/workspace/test/packages/hands/allegro_hand/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
- link link_7.0: geometry collision box size=0.0196 0.0269 0.022; visual mesh filename=/home/wangminqi/workspace/test/packages/hands/allegro_hand/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
- link link_7.0_tip: geometry collision mesh filename=/home/wangminqi/workspace/test/packages/hands/allegro_hand/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; visual mesh filename=/home/wangminqi/workspace/test/packages/hands/allegro_hand/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
- link link_8.0: geometry collision box size=0.0196 0.0275 0.0164; visual mesh filename=/home/wangminqi/workspace/test/packages/hands/allegro_hand/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
- link link_9.0: geometry collision box size=0.0196 0.0275 0.054; visual mesh filename=/home/wangminqi/workspace/test/packages/hands/allegro_hand/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

File: retarget_wmq/urdf/inspire_hand_right_glb.urdf (robot description, URDF)
Before this commit: robot inspire_hand_right, 25 links, 24 joints
Links:
- link hand_base_link: geometry collision box size=0.0125 0.0111 0.0089; collision box size=0.0125 0.0111 0.0089
- link index_intermediate: geometry collision mesh filename=/home/wangminqi/workspace/test/packages/hands/inspire_hand/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; visual mesh filename=/home/wangminqi/workspace/test/packages/hands/inspire_hand/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
- link index_proximal: geometry collision mesh filename=/home/wangminqi/workspace/test/packages/hands/inspire_hand/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; visual mesh filename=/home/wangminqi/workspace/test/packages/hands/inspire_hand/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
- link middle_intermediate: geometry collision mesh filename=/home/wangminqi/workspace/test/packages/hands/inspire_hand/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; visual mesh filename=/home/wangminqi/workspace/test/packages/hands/inspire_hand/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
- link middle_proximal: geometry collision mesh filename=/home/wangminqi/workspace/test/packages/hands/inspire_hand/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; visual mesh filename=/home/wangminqi/workspace/test/packages/hands/inspire_hand/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
- link pinky_intermediate: geometry collision mesh filename=/home/wangminqi/workspace/test/packages/hands/inspire_hand/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; visual mesh filename=/home/wangminqi/workspace/test/packages/hands/inspire_hand/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
- link pinky_proximal: geometry collision mesh filename=/home/wangminqi/workspace/test/packages/hands/inspire_hand/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; visual mesh filename=/home/wangminqi/workspace/test/packages/hands/inspire_hand/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
- link ring_intermediate: geometry collision mesh filename=/home/wangminqi/workspace/test/packages/hands/inspire_hand/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; visual mesh filename=/home/wangminqi/workspace/test/packages/hands/inspire_hand/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
- link ring_proximal: geometry collision mesh filename=/home/wangminqi/workspace/test/packages/hands/inspire_hand/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; visual mesh filename=/home/wangminqi/workspace/test/packages/hands/inspire_hand/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
- link thumb_distal: geometry collision mesh filename=/home/wangminqi/workspace/test/packages/hands/inspire_hand/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; visual mesh filename=/home/wangminqi/workspace/test/packages/hands/inspire_hand/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
- link thumb_intermediate: geometry collision mesh filename=/home/wangminqi/workspace/test/packages/hands/inspire_hand/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; visual mesh filename=/home/wangminqi/workspace/test/packages/hands/inspire_hand/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
- link thumb_proximal: geometry collision mesh filename=/home/wangminqi/workspace/test/packages/hands/inspire_hand/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; visual mesh filename=/home/wangminqi/workspace/test/packages/hands/inspire_hand/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
- link thumb_proximal_base: geometry collision mesh filename=/home/wangminqi/workspace/test/packages/hands/inspire_hand/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; visual mesh filename=/home/wangminqi/workspace/test/packages/hands/inspire_hand/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

File: retarget_wmq/urdf/leap_hand_left_glb.urdf (robot description, URDF)
Before this commit: robot leap_left, 28 links, 27 joints
Links:
- link dip: geometry collision box size=0.014 0.02 0.004; collision box size=0.014 0.02 0.004
- link dip_2: geometry collision box size=0.014 0.02 0.004; collision box size=0.014 0.02 0.004
- link dip_3: geometry collision box size=0.014 0.02 0.004; collision box size=0.014 0.02 0.004
- link fingertip: geometry collision box size=0.014 0.022 0.004; collision box size=0.014 0.022 0.004
- link fingertip_2: geometry collision box size=0.014 0.022 0.004; collision box size=0.014 0.022 0.004
- link fingertip_3: geometry collision box size=0.014 0.022 0.004; collision box size=0.014 0.022 0.004
- link mcp_joint: geometry collision box size=0.014 0.02 0.004; collision box size=0.014 0.02 0.004
- link mcp_joint_2: geometry collision box size=0.014 0.02 0.004; collision box size=0.014 0.02 0.004
- link mcp_joint_3: geometry collision box size=0.014 0.02 0.004; collision box size=0.014 0.02 0.004
- link palm_lower_left: geometry collision box size=0.004 0.036 0.034; collision box size=0.01 0.12 0.02
- link pip: geometry collision box size=0.034 0.026 0.022; visual mesh filename=/home/wangminqi/workspace/test/packages/hands/leap_hand/mes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
- link pip_2: geometry collision box size=0.034 0.026 0.022; visual mesh filename=/home/wangminqi/workspace/test/packages/hands/leap_hand/mes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
- link pip_3: geometry collision box size=0.034 0.026 0.022; visual mesh filename=/home/wangminqi/workspace/test/packages/hands/leap_hand/mes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
- link thumb_dip: geometry collision box size=0.01 0.024 0.018; collision box size=0.014 0.02 0.004
- link thumb_fingertip: geometry collision box size=0.008 0.024 0.018; collision box size=0.02 0.004 0.03
- link thumb_left_temp_base: geometry collision box size=0.034 0.026 0.022; visual mesh filename=/home/wangminqi/workspace/test/packages/hands/leap_hand/mes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
- link thumb_pip: geometry collision box size=0.014 0.004 0.02; collision box size=0.014 0.004 0.02

File: retarget_wmq/urdf/leap_hand_right_glb.urdf (robot description, URDF)
Before this commit: robot leap_right, 28 links, 27 joints
Links:
- link dip: geometry collision box size=0.014 0.02 0.004; collision box size=0.014 0.02 0.004
- link dip_2: geometry collision box size=0.014 0.02 0.004; collision box size=0.014 0.02 0.004
- link dip_3: geometry collision box size=0.014 0.02 0.004; collision box size=0.014 0.02 0.004
- link fingertip: geometry collision box size=0.014 0.022 0.004; collision box size=0.014 0.022 0.004
- link fingertip_2: geometry collision box size=0.014 0.022 0.004; collision box size=0.014 0.022 0.004
- link fingertip_3: geometry collision box size=0.014 0.022 0.004; collision box size=0.014 0.022 0.004
- link mcp_joint: geometry collision box size=0.014 0.02 0.004; collision box size=0.014 0.02 0.004
- link mcp_joint_2: geometry collision box size=0.014 0.02 0.004; collision box size=0.014 0.02 0.004
- link mcp_joint_3: geometry collision box size=0.014 0.02 0.004; collision box size=0.014 0.02 0.004
- link palm_lower: geometry collision box size=0.004 0.036 0.034; collision box size=0.01 0.12 0.02
- link pip: geometry collision box size=0.034 0.026 0.022; visual mesh filename=/home/wangminqi/workspace/test/packages/hands/leap_hand/mes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
- link pip_2: geometry collision box size=0.034 0.026 0.022; visual mesh filename=/home/wangminqi/workspace/test/packages/hands/leap_hand/mes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
- link pip_3: geometry collision box size=0.034 0.026 0.022; visual mesh filename=/home/wangminqi/workspace/test/packages/hands/leap_hand/mes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
- link thumb_dip: geometry collision box size=0.01 0.024 0.018; collision box size=0.014 0.02 0.004
- link thumb_fingertip: geometry collision box size=0.008 0.024 0.018; collision box size=0.02 0.004 0.03
- link thumb_pip: geometry collision box size=0.014 0.004 0.02; collision box size=0.014 0.004 0.02
- link thumb_temp_base: geometry collision box size=0.034 0.026 0.022; visual mesh filename=/home/wangminqi/workspace/test/packages/hands/leap_hand/mes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

File: retarget_wmq/urdf/shadow_hand_left_glb.urdf (robot description, URDF)
Before this commit: robot shadow_left, 39 links, 38 joints
Links:
- link ffdistal: geometry collision mesh filename=/home/wangminqi/workspace/test/packages/hands/shadow_hand/m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 scale=0.001 0.001 0.001; visual mesh filename=/home/wangminqi/workspace/test/packages/hands/shadow_hand/m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 scale=0.001 0.001 0.001
- link ffknuckle: geometry collision mesh filename=/home/wangminqi/workspace/test/packages/hands/shadow_hand/m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; visual mesh filename=/home/wangminqi/workspace/test/packages/hands/shadow_hand/m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 scale=0.001 0.001 0.001
- link ffmiddle: geometry collision cylinder length=0.025 radius=0.007; collision sphere radius=0.007
- link ffproximal: geometry collision cylinder length=0.04 radius=0.007; visual mesh filename=/home/wangminqi/workspace/test/packages/hands/shadow_hand/m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 scale=0.001 0.001 0.001
- link forearm: geometry collision box size=0.07 0.07 0.07; collision mesh filename=/home/wangminqi/workspace/test/packages/hands/shadow_hand/m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 scale=0.001 0.001 0.001
- link lfdistal: geometry collision mesh filename=/home/wangminqi/workspace/test/packages/hands/shadow_hand/m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 scale=0.001 0.001 0.001; visual mesh filename=/home/wangminqi/workspace/test/packages/hands/shadow_hand/m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 scale=0.001 0.001 0.001
- link lfknuckle: geometry collision mesh filename=/home/wangminqi/workspace/test/packages/hands/shadow_hand/m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; visual mesh filename=/home/wangminqi/workspace/test/packages/hands/shadow_hand/m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 scale=0.001 0.001 0.001
- link lfmetacarpal: geometry collision box size=0.018 0.024 0.04; visual mesh filename=/home/wangminqi/workspace/test/packages/hands/shadow_hand/m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 scale=0.001 0.001 0.001
- link lfmiddle: geometry collision cylinder length=0.025 radius=0.007; collision sphere radius=0.007
- link lfproximal: geometry collision cylinder length=0.04 radius=0.007; visual mesh filename=/home/wangminqi/workspace/test/packages/hands/shadow_hand/m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 scale=0.001 0.001 0.001
- link mfdistal: geometry collision mesh filename=/home/wangminqi/workspace/test/packages/hands/shadow_hand/m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 scale=0.001 0.001 0.001; visual mesh filename=/home/wangminqi/workspace/test/packages/hands/shadow_hand/m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 scale=0.001 0.001 0.001
- link mfknuckle: geometry collision mesh filename=/home/wangminqi/workspace/test/packages/hands/shadow_hand/m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; visual mesh filename=/home/wangminqi/workspace/test/packages/hands/shadow_hand/m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 scale=0.001 0.001 0.001
- link mfmiddle: geometry collision cylinder length=0.025 radius=0.007; collision sphere radius=0.007
- link mfproximal: geometry collision cylinder length=0.04 radius=0.007; visual mesh filename=/home/wangminqi/workspace/test/packages/hands/shadow_hand/m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 scale=0.001 0.001 0.001
- link palm: geometry collision box size=0.018 0.024 0.004; collision box size=0.02 0.024 0.032
- link rfdistal: geometry collision mesh filename=/home/wangminqi/workspace/test/packages/hands/shadow_hand/m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 scale=0.001 0.001 0.001; visual mesh filename=/home/wangminqi/workspace/test/packages/hands/shadow_hand/m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 scale=0.001 0.001 0.001
- link rfknuckle: geometry collision mesh filename=/home/wangminqi/workspace/test/packages/hands/shadow_hand/m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; visual mesh filename=/home/wangminqi/workspace/test/packages/hands/shadow_hand/m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 scale=0.001 0.001 0.001
- link rfmiddle: geometry collision cylinder length=0.025 radius=0.007; collision sphere radius=0.007
- link rfproximal: geometry collision cylinder length=0.04 radius=0.007; visual mesh filename=/home/wangminqi/workspace/test/packages/hands/shadow_hand/m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 scale=0.001 0.001 0.001
- link thdistal: geometry collision mesh filename=/home/wangminqi/workspace/test/packages/hands/shadow_hand/m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 scale=0.001 0.001 0.001; visual mesh filename=/home/wangminqi/workspace/test/packages/hands/shadow_hand/m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 scale=0.001 0.001 0.001
- link thmiddle: geometry collision mesh filename=/home/wangminqi/workspace/test/packages/hands/shadow_hand/m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 scale=0.001 0.001 0.001; visual mesh filename=/home/wangminqi/workspace/test/packages/hands/shadow_hand/m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 scale=0.001 0.001 0.001
- link thproximal: geometry collision mesh filename=/home/wangminqi/workspace/test/packages/hands/shadow_hand/m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 scale=0.001 0.001 0.001; visual mesh filename=/home/wangminqi/workspace/test/packages/hands/shadow_hand/m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 scale=0.001 0.001 0.001
- link wrist: geometry collision box size=0.027 0.018 0.01; collision box size=0.027 0.018 0.01

File: retarget_wmq/urdf/shadow_hand_right_glb.urdf (robot description, URDF)
Before this commit: robot shadow_right, 39 links, 38 joints
Links:
- link ffdistal: geometry collision mesh filename=/home/wangminqi/workspace/test/packages/hands/shadow_hand/m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 scale=0.001 0.001 0.001; visual mesh filename=/home/wangminqi/workspace/test/packages/hands/shadow_hand/m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 scale=0.001 0.001 0.001
- link ffknuckle: geometry collision mesh filename=/home/wangminqi/workspace/test/packages/hands/shadow_hand/m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; visual mesh filename=/home/wangminqi/workspace/test/packages/hands/shadow_hand/m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 scale=0.001 0.001 0.001
- link ffmiddle: geometry collision cylinder length=0.025 radius=0.007; collision sphere radius=0.007
- link ffproximal: geometry collision cylinder length=0.04 radius=0.007; visual mesh filename=/home/wangminqi/workspace/test/packages/hands/shadow_hand/m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 scale=0.001 0.001 0.001
- link forearm: geometry collision box size=0.07 0.07 0.07; collision mesh filename=/home/wangminqi/workspace/test/packages/hands/shadow_hand/m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 scale=0.001 0.001 0.001
- link lfdistal: geometry collision mesh filename=/home/wangminqi/workspace/test/packages/hands/shadow_hand/m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 scale=0.001 0.001 0.001; visual mesh filename=/home/wangminqi/workspace/test/packages/hands/shadow_hand/m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 scale=0.001 0.001 0.001
- link lfknuckle: geometry collision mesh filename=/home/wangminqi/workspace/test/packages/hands/shadow_hand/m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; visual mesh filename=/home/wangminqi/workspace/test/packages/hands/shadow_hand/m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 scale=0.001 0.001 0.001
- link lfmetacarpal: geometry collision box size=0.018 0.024 0.04; visual mesh filename=/home/wangminqi/workspace/test/packages/hands/shadow_hand/m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 scale=0.001 0.001 0.001
- link lfmiddle: geometry collision cylinder length=0.025 radius=0.007; collision sphere radius=0.007
- link lfproximal: geometry collision cylinder length=0.04 radius=0.007; visual mesh filename=/home/wangminqi/workspace/test/packages/hands/shadow_hand/m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 scale=0.001 0.001 0.001
- link mfdistal: geometry collision mesh filename=/home/wangminqi/workspace/test/packages/hands/shadow_hand/m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 scale=0.001 0.001 0.001; visual mesh filename=/home/wangminqi/workspace/test/packages/hands/shadow_hand/m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 scale=0.001 0.001 0.001
- link mfknuckle: geometry collision mesh filename=/home/wangminqi/workspace/test/packages/hands/shadow_hand/m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; visual mesh filename=/home/wangminqi/workspace/test/packages/hands/shadow_hand/m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 scale=0.001 0.001 0.001
- link mfmiddle: geometry collision cylinder length=0.025 radius=0.007; collision sphere radius=0.007
- link mfproximal: geometry collision cylinder length=0.04 radius=0.007; visual mesh filename=/home/wangminqi/workspace/test/packages/hands/shadow_hand/m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 scale=0.001 0.001 0.001
- link palm: geometry collision box size=0.018 0.024 0.004; collision box size=0.02 0.024 0.032
- link rfdistal: geometry collision mesh filename=/home/wangminqi/workspace/test/packages/hands/shadow_hand/m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 scale=0.001 0.001 0.001; visual mesh filename=/home/wangminqi/workspace/test/packages/hands/shadow_hand/m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 scale=0.001 0.001 0.001
- link rfknuckle: geometry collision mesh filename=/home/wangminqi/workspace/test/packages/hands/shadow_hand/m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; visual mesh filename=/home/wangminqi/workspace/test/packages/hands/shadow_hand/m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 scale=0.001 0.001 0.001
- link rfmiddle: geometry collision cylinder length=0.025 radius=0.007; collision sphere radius=0.007
- link rfproximal: geometry collision cylinder length=0.04 radius=0.007; visual mesh filename=/home/wangminqi/workspace/test/packages/hands/shadow_hand/m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 scale=0.001 0.001 0.001
- link thdistal: geometry collision mesh filename=/home/wangminqi/workspace/test/packages/hands/shadow_hand/m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 scale=0.001 0.001 0.001; visual mesh filename=/home/wangminqi/workspace/test/packages/hands/shadow_hand/m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 scale=0.001 0.001 0.001
- link thmiddle: geometry collision mesh filename=/home/wangminqi/workspace/test/packages/hands/shadow_hand/m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 scale=0.001 0.001 0.001; visual mesh filename=/home/wangminqi/workspace/test/packages/hands/shadow_hand/m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 scale=0.001 0.001 0.001
- link thproximal: geometry collision mesh filename=/home/wangminqi/workspace/test/packages/hands/shadow_hand/m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 scale=0.001 0.001 0.001; visual mesh filename=/home/wangminqi/workspace/test/packages/hands/shadow_hand/m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 scale=0.001 0.001 0.001
- link wrist: geometry collision box size=0.027 0.018 0.01; collision box size=0.027 0.018 0.01
